File: final_project/TECHIN514_w26_project_PCB_Peizhong_Gao/TECHIN514_w26_project_PCB_Peizhong_Gao.kicad_sch (KiCad schematic)
At the start: 12 parts, among them M1 Stepper_Motor_unipolar_5pin, SW1 SW_Push, SW3 SW_Push, U1 MOUDLE-SEEEDUINO-XIAO-ESP32C3, U2 PIR adafruit, U3 MAX9814, U4 MOUDLE-SEEEDUINO-XIAO-ESP32C3, U5 ULN2003APG

Commit message: 0126-new
Connections:
- net IN1: now reaches U4.2 (PA4_A1_D1)
- net IN1: now also M1.2, U5.2 (IN1)
- net IN2: now reaches U4.3 (PA10_A2_D2)
- net IN2: now also M1.3 (-), U5.3 (IN2)
- net IN3: now reaches U4.4 (PA11_A3_D3)
- net IN3: now also M1.4, U5.4 (IN3)
- net IN4: now reaches U4.5 (PA8_A4_D4_SDA)
- net IN4: now also M1.5, U5.5 (IN4)
Other:
- moved on the sheet: U5

Commit message: 0126-new2
Connections:
- net GND: now also U4.13 (GND)
Changed lines of the file:
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@@
 	(paper "A4")
+	(junction
+		(at 146.05 104.14)
+		(diameter 0)
+		(color 0 0 0 0)
+	)
 	(junction
 		(at 147.32 49.53)
@@
 		)
 		(stroke
+			(width 0)
+			(type default)
+		)
+	)
+	(wire
+		(pts
+			(xy 121.92 104.14) (xy 146.05 104.14)
+		)
+		(stroke
